Commit message: distance 0.5 for perfect timing

File: urdf/dual_ur5e.urdf.xacro (robot description, xacro)
@@ -39,3 +39,22 @@
     <origin xyz="1 0 0" rpy="0 0 0"/>
   </xacro:ur_robot>
+  <!-- ============================== -->
+  <!-- Inner-side safety sensor frames -->
+  <!-- ============================== -->
+  <!--
+    Both sensors use identical offsets to maintain the same orientation.
+    Robot 1 and Robot 2 both face the same direction (Z rotation = 0).
+  -->
+  <link name="robot1_inner_sensor"/>
+  <joint name="robot1_inner_sensor_joint" type="fixed">
+    <parent link="robot1_tool0"/>
+    <child link="robot1_inner_sensor"/>
+    <origin xyz="0 0.10 0" rpy="0 0 0"/>
+  </joint>
+  <link name="robot2_inner_sensor"/>
+  <joint name="robot2_inner_sensor_joint" type="fixed">
+    <parent link="robot2_tool0"/>
+    <child link="robot2_inner_sensor"/>
+    <origin xyz="0 0.10 0" rpy="0 0 0"/>
+  </joint>
 </robot>

Commit message: final version

File: urdf/dual_ur5e.urdf.xacro (robot description, xacro)
@@ -37,5 +37,6 @@
     generate_ros2_control_tag="true"
   >
-    <origin xyz="1 0 0" rpy="0 0 0"/>
+    <!-- Base rotated 180° so Robot 2 faces Robot 1 from spawn — no runtime pan spin needed -->
+    <origin xyz="1 0 0" rpy="0 0 3.14159"/>
   </xacro:ur_robot>
   <!-- ============================== -->
